File: Hardware/PCB.brd (EAGLE design)
At the start: 46 x 35 mm, 105 parts, among them IC1 BQ25180YBGR, IC2 DRV2605YZFR, IC3 BMA423, IC9 RT6160AWSC, J1 503480-2400, J2 TC2030-IDC, J4 KH-TYPE-C-16P, Q3 SI1308EDL-T1-GE3, U1 NRF52840_QF, U3 MAX17048G+T10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

Commit message: Add files via upload
Parts:
- moved ANT1 1.55 mm to (63.7, 143.4), turned to 90 degrees
- moved C11 0.66 mm to (57.7, 129.2)
Routing:
- net GND: track 64.9 -> 65.6 mm
Other:
- board size 46 x 35 mm -> 46 x 35.1 mm
